File: CAD/KiCAD/SSR_4CH.sch (KiCad schematic (older format))
At the start: 4 parts, among them K1 G3MB202PDC12, K2 G3MB202PDC12, K3 G3MB202PDC12, K4 G3MB202PDC12

Commit message: Using A0 instead of A3 now.
Parts:
- K1, K2, K3, K4: symbol Schematic-rescue:G3MB202PDC12-BhallaLabComponents -> Schematic-rescue:G3MB202PDC12-BhallaLabComponents-Schematic-rescue
Changed lines of the file:
@@
 $EndDescr
 $Comp
-L Schematic-rescue:G3MB202PDC12-BhallaLabComponents K2
+L Schematic-rescue:G3MB202PDC12-BhallaLabComponents-Schematic-rescue K2
 U 1 1 5D18AD83
 P 5225 3975
@@
 	5725 4125 5740 4125
 $Comp
-L Schematic-rescue:G3MB202PDC12-BhallaLabComponents K1
+L Schematic-rescue:G3MB202PDC12-BhallaLabComponents-Schematic-rescue K1
 U 1 1 5D18ADB3
 P 4575 3975
@@
 Connection ~ 4900 3225
 $Comp
-L Schematic-rescue:G3MB202PDC12-BhallaLabComponents K3
+L Schematic-rescue:G3MB202PDC12-BhallaLabComponents-Schematic-rescue K3
 U 1 1 5D1D4113
 P 5950 3975
@@
 $EndComp
 $Comp
-L Schematic-rescue:G3MB202PDC12-BhallaLabComponents K4
+L Schematic-rescue:G3MB202PDC12-BhallaLabComponents-Schematic-rescue K4
 U 1 1 5D1D5B7E
 P 6800 3975

Commit message: Passing electrical rules.
Parts:
- K1, K2, K3, K4: symbol Schematic-rescue:G3MB202PDC12-BhallaLabComponents-Schematic-rescue -> Schematic-rescue:G3MB202PDC12-BhallaLabComponents-Schematic-rescue-Schematic-rescue
Changed lines of the file:
@@
 $EndDescr
 $Comp
-L Schematic-rescue:G3MB202PDC12-BhallaLabComponents-Schematic-rescue K2
+L Schematic-rescue:G3MB202PDC12-BhallaLabComponents-Schematic-rescue-Schematic-rescue K2
 U 1 1 5D18AD83
 P 5225 3975
+AR Path="/5D18AD83" Ref="K2"  Part="1"
+AR Path="/5D1ADABF/5D18AD83" Ref="K2"  Part="1"
 F 0 "K2" V 4460 4045 50  0000 C CNN
 F 1 "G3MB202PDC12" V 4551 4045 50  0000 C CNN
@@
 	5725 4125 5740 4125
 $Comp
-L Schematic-rescue:G3MB202PDC12-BhallaLabComponents-Schematic-rescue K1
+L Schematic-rescue:G3MB202PDC12-BhallaLabComponents-Schematic-rescue-Schematic-rescue K1
 U 1 1 5D18ADB3
 P 4575 3975
+AR Path="/5D18ADB3" Ref="K1"  Part="1"
+AR Path="/5D1ADABF/5D18ADB3" Ref="K1"  Part="1"
 F 0 "K1" V 3810 4045 50  0000 C CNN
 F 1 "G3MB202PDC12" V 3901 4045 50  0000 C CNN
@@
 Connection ~ 4900 3225
 $Comp
-L Schematic-rescue:G3MB202PDC12-BhallaLabComponents-Schematic-rescue K3
+L Schematic-rescue:G3MB202PDC12-BhallaLabComponents-Schematic-rescue-Schematic-rescue K3
 U 1 1 5D1D4113
 P 5950 3975
+AR Path="/5D1D4113" Ref="K3"  Part="1"
+AR Path="/5D1ADABF/5D1D4113" Ref="K3"  Part="1"
 F 0 "K3" V 5185 4045 50  0000 C CNN
 F 1 "G3MB202PDC12" V 5276 4045 50  0000 C CNN
@@
 $EndComp
 $Comp
-L Schematic-rescue:G3MB202PDC12-BhallaLabComponents-Schematic-rescue K4
+L Schematic-rescue:G3MB202PDC12-BhallaLabComponents-Schematic-rescue-Schematic-rescue K4
 U 1 1 5D1D5B7E
 P 6800 3975
+AR Path="/5D1D5B7E" Ref="K4"  Part="1"
+AR Path="/5D1ADABF/5D1D5B7E" Ref="K4"  Part="1"
 F 0 "K4" V 6035 4045 50  0000 C CNN
 F 1 "G3MB202PDC12" V 6126 4045 50  0000 C CNN
