File: CAD/KiCAD/Schematic.sch (KiCad schematic (older format))
At the start: 8 parts, among them U1 4N35

Commit message: Using A0 instead of A3 now.
Parts:
- RotaryEncoder1: symbol Schematic-rescue:RotaryEncoder-OrangeRotaryEncoder-Schematic-rescue -> Schematic-rescue:RotaryEncoder-OrangeRotaryEncoder-Schematic-rescue-Schematic-rescue
- ShockPad1: symbol Schematic-rescue:ShockPad-BhallaLabComponents-Schematic-rescue -> Schematic-rescue:ShockPad-BhallaLabComponents-Schematic-rescue-Schematic-rescue
Connections:
- wire segments 77 -> 78
Changed lines of the file:
@@
 $EndComp
 $Comp
-L Schematic-rescue:RotaryEncoder-OrangeRotaryEncoder-Schematic-rescue RotaryEncoder1
+L Schematic-rescue:RotaryEncoder-OrangeRotaryEncoder-Schematic-rescue-Schematic-rescue RotaryEncoder1
 U 1 1 5D191567
 P 2750 2450
@@
 	4175 3050 4175 4175
 Wire Wire Line
-	5600 3250 5400 3250
-Wire Wire Line
 	4175 4175 5100 4175
 Wire Wire Line
@@
 Wire Wire Line
 	5850 3250 5600 3250
-Connection ~ 5600 3250
 Text Notes 3700 4250 0    50   ~ 0
 D5, PWM, 20 kHz
@@
 PAD+
 $Comp
-L Schematic-rescue:ShockPad-BhallaLabComponents-Schematic-rescue ShockPad1
+L Schematic-rescue:ShockPad-BhallaLabComponents-Schematic-rescue-Schematic-rescue ShockPad1
 U 1 1 5D197A8E
 P 8425 3775
@@
 Text Notes 5800 3100 0    50   ~ 0
 When paw is on shockpad\ntau should be approx 1ms.
+Wire Wire Line
+	5850 3250 5850 2950
+Wire Wire Line
+	5850 2950 5400 2950
 $EndSCHEMATC

Commit message: Passing electrical rules.
Parts:
- removed ArduinoUno1: Arduino_UNO_R3, Module:Arduino_UNO_R3, symbol MCU_Module:Arduino_UNO_R3
- removed CA3: 47nF, symbol Device:C
- removed D1: LED, symbol Device:LED
- removed LS1: Speaker, symbol Device:Speaker
- removed RA3: 10K-1M, symbol Device:R_Variable
- removed RotaryEncoder1: RotaryEncoder, symbol Schematic-rescue:RotaryEncoder-OrangeRotaryEncoder-Schematic-rescue-Schematic-r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
- removed ShockPad1: ShockPad, symbol Schematic-rescue:ShockPad-BhallaLabComponents-Schematic-rescue-Schematic-rescue
- removed U1: 4N35, Package_DIP:DIP-6_W7.62mm, symbol Isolator:4N35
- added C1: 47 uF, Capacitor_THT:CP_Axial_L11.0mm_D6.0mm_P18.00mm_Horizontal, symbol Device:C
- added CN1: OutputPad, Connector_PinHeader_2.54mm:PinHeader_1x15_P2.54mm_Horizontal, symbol ArduinoEncoderShield_old-rescue:HDR-1X15-15-91-?
- added D1: DIODE, Diode_THT:D_5KP_P12.70mm_Horizontal, symbol ArduinoEncoderShield_old-rescue:DIODE
- added IC1, IC2, IC3, IC4, IC5: 4N35, Package_DIP:DIP-6_W7.62mm_Socket, symbol Isolator:4N35
- added J-InStimInput1: 90V, Connector_BarrelJack:BarrelJack_CUI_PJ-036AH-SMT_Horizontal, symbol Connector:Jack-DC
- added J1: SSR-ToInput, Connector_PinSocket_2.54mm:PinSocket_1x06_P2.54mm_Vertical, symbol Connector_Generic:Conn_01x06
- added J2: SSR-ToOutput, symbol Connector_Generic:Conn_01x08
- added JPad1: ShockPad, TerminalBlock:TerminalBlock_Altech_AK300-2_P5.00mm, symbol Connector:Screw_Terminal_01x02
- added JPad2: StimInput, TerminalBlock:TerminalBlock_Altech_AK300-2_P5.00mm, symbol Connector:Screw_Terminal_01x02
- added P1, P2: CONN_6, Connector_PinHeader_1.27mm:PinHeader_1x06_P1.27mm_Horizontal, symbol ArduinoEncoderShield_old-rescue:CONN_6
- added P4: CONN_2, Connector_PinHeader_1.27mm:PinHeader_1x02_P1.27mm_Vertical, symbol ArduinoEncoderShield_old-rescue:CONN_2
- added P7: CONN_2, symbol ArduinoEncoderShield_old-rescue:CONN_2
- added P8, P9: CONN_8, Connector_PinHeader_1.27mm:PinHeader_1x08_P1.27mm_Horizontal, symbol ArduinoEncoderShield_old-rescue:CONN_8
- added R1, R2: 560E, Resistor_SMD:R_0603_1608Metric_Pad1.05x0.95mm_HandSolder, symbol ArduinoEncoderShield_old-rescue:R
- added R10, R12, R4: 560E, Resistor_SMD:R_0805_2012Metric_Pad1.15x1.40mm_HandSolder, symbol ArduinoEncoderShield_old-rescue:R
- added R11, R13, R7, R8, R9: 15k, Resistor_SMD:R_0805_2012Metric_Pad1.15x1.40mm_HandSolder, symbol ArduinoEncoderShield_old-rescue:R
- added R3: 10k-1M, Potentiometer_THT:Potentiometer_Alps_RK09K_Single_Vertical, symbol Device:R_Variable
- added R5, R6: 470E, Resistor_SMD:R_0805_2012Metric_Pad1.15x1.40mm_HandSolder, symbol ArduinoEncoderShield_old-rescue:R
- added SHIELD1: ARDUINO_SHIELD, symbol ArduinoEncoderShield_old-rescue:ARDUINO_SHIELD
- added U1: ULN2003A, Package_DIP:DIP-16_W7.62mm_Socket, symbol ArduinoEncoderShield_old-rescue:ULN2003A
Connections:
- net labels added: 12 V, 5V, A0, A1, A2, A3, A4, A5, AGND, D0, D1, D10, D11, D12, D13, D2, D3, D4, D5, D6, D7, D8, D9, DGND, EX 5 V, RST, Solenoid1_1, Solenoid1_2, Solenoid2_1, Solenoid2_2, Spare1, Spare2, Tone1, Tone2, Tone3, ULN_IN1, ULN_IN2
- net labels removed: CAM, GND, IMAGING_TRIG, LED, PAD+, PAD-, PUFF, TONE, VCC
- wire segments 78 -> 91
- no-connect marks 0 -> 23
Other:
- note added: "SolenoidDrivers\n"
- note added: "ToneDrivers\n"
- note removed: "1200 counts per cycle."
- note removed: "CH1=CH2 \nCH3=CH4=~CH1\nImplemented in Arduino."
- note removed: "D5, PWM, 20 kHz"
- note removed: "Low Level Trigger.\nVendor: NA \nAsk hrishi@ncbs.res.in"
- note removed: "Not implemented.\nUsing as black-box."
- note removed: "Resistance of mouse's paw is of the order of 1M.\nThe value of R2 must be the same."
- note removed: "To solenoid."
- note removed: "When paw is on shockpad\ntau should be approx 1ms."

Commit message: refactoring.
Parts:
- CN1: symbol ArduinoEncoderShield_old-rescue:HDR-1X15-15-91-? -> Dorababu:HDR-1X15-15-91-?
- D1: symbol ArduinoEncoderShield_old-rescue:DIODE -> Dorababu:DIODE
- P1, P2: symbol ArduinoEncoderShield_old-rescue:CONN_6 -> Dorababu:CONN_6
- P4, P7: symbol ArduinoEncoderShield_old-rescue:CONN_2 -> Dorababu:CONN_2
- P8, P9: symbol ArduinoEncoderShield_old-rescue:CONN_8 -> Dorababu:CONN_8
- R1, R10, R11, R12, R13, R2, R4, R5, R6, R7, R8, R9: symbol ArduinoEncoderShield_old-rescue:R -> Dorababu:R
- SHIELD1: symbol ArduinoEncoderShield_old-rescue:ARDUINO_SHIELD -> DoraBabu:ARDUINO_SHIELD
- U1: symbol ArduinoEncoderShield_old-rescue:ULN2003A -> Dorababu:ULN2003A
Changed lines of the file:
@@
 EESchema Schematic File Version 4
-LIBS:ArduinoEncoderShield_old-cache
 EELAYER 29 0
 EELAYER END
@@
 $EndComp
 $Comp
-L ArduinoEncoderShield_old-rescue:ULN2003A U1
+L Dorababu:ULN2003A U1
 U 1 1 5C3EFA71
 P 9300 1225
@@
 $EndComp
 $Comp
-L ArduinoEncoderShield_old-rescue:DIODE D1
+L Dorababu:DIODE D1
 U 1 1 5C3EFA72
 P 10300 1625
@@
 $EndComp
 $Comp
-L ArduinoEncoderShield_old-rescue:R R8
+L Dorababu:R R8
 U 1 1 5C3EFA76
 P 7575 2200
@@
 $EndComp
 $Comp
-L ArduinoEncoderShield_old-rescue:R R6
+L Dorababu:R R6
 U 1 1 5C3EFA82
 P 6575 1700
@@
 $EndComp
 $Comp
-L ArduinoEncoderShield_old-rescue:R R5
+L Dorababu:R R5
 U 1 1 5C3EFA83
 P 6575 700
@@
 $EndComp
 $Comp
-L ArduinoEncoderShield_old-rescue:R R10
+L Dorababu:R R10
 U 1 1 5C3EFA84
 P 7925 5425
@@
 12 V
 $Comp
-L ArduinoEncoderShield_old-rescue:CONN_8 P8
+L Dorababu:CONN_8 P8
 U 1 1 5C3EFA87
 P 3475 5100
@@
 $EndComp
 $Comp
-L ArduinoEncoderShield_old-rescue:CONN_6 P2
+L Dorababu:CONN_6 P2
 U 1 1 5C3EFA88
 P 950 1800
@@
 Solenoid2_2
 $Comp
-L ArduinoEncoderShield_old-rescue:HDR-1X15-15-91-? CN1
+L Dorababu:HDR-1X15-15-91-? CN1
 U 1 1 5C3EFA8D
 P 1650 5500
@@
 $EndComp
 $Comp
-L ArduinoEncoderShield_old-rescue:R R12
+L Dorababu:R R12
 U 1 1 5C3EFA8E
 P 9825 5425
@@
 Tone2
 $Comp
-L ArduinoEncoderShield_old-rescue:R R4
+L Dorababu:R R4
 U 1 1 5C3EFA94
 P 5975 5425
@@
 EX 5 V
 $Comp
-L ArduinoEncoderShield_old-rescue:R R7
+L Dorababu:R R7
 U 1 1 5C3EFA96
 P 6975 5925
@@
 Connection ~ 10050 1875
 $Comp
-L ArduinoEncoderShield_old-rescue:R R1
+L Dorababu:R R1
 U 1 1 5C3EFA99
 P 2550 4100
@@
 $EndComp
 $Comp
-L ArduinoEncoderShield_old-rescue:R R2
+L Dorababu:R R2
 U 1 1 5C3EFA9A
 P 2550 4300
@@
 $EndComp
 $Comp
-L ArduinoEncoderShield_old-rescue:CONN_2 P7
+L Dorababu:CONN_2 P7
 U 1 1 5C3EFA9B
 P 3200 4200
@@
 D11
 $Comp
-L ArduinoEncoderShield_old-rescue:CONN_8 P9
+L Dorababu:CONN_8 P9
 U 1 1 5C3EFD0C
 P 3475 6100
@@
 Connection ~ 6975 5625
 $Comp
-L ArduinoEncoderShield_old-rescue:CONN_6 P1
+L Dorababu:CONN_6 P1
 U 1 1 5C3F096C
 P 950 1100
@@
 EX 5 V
 $Comp
-L ArduinoEncoderShield_old-rescue:R R11
+L Dorababu:R R11
 U 1 1 5C3F0A84
 P 8875 5975
@@
 	8875 5725 8875 5675
 $Comp
-L ArduinoEncoderShield_old-rescue:AGND #PWR05
+L Dorababu:AGND #PWR05
 U 1 1 5C3F0AE2
 P 8875 6325
@@
 DGND
 $Comp
-L ArduinoEncoderShield_old-rescue:R R13
+L Dorababu:R R13
 U 1 1 5C3F0BA2
 P 10775 5975
@@
 $EndComp
 $Comp
-L ArduinoEncoderShield_old-rescue:AGND #PWR07
+L Dorababu:AGND #PWR07
 U 1 1 5C3F0BA8
 P 10775 6325
@@
 AGND
 $Comp
-L ArduinoEncoderShield_old-rescue:AGND #PWR02
+L Dorababu:AGND #PWR02
 U 1 1 5C3F0CE1
 P 6975 6225
@@
 AGND
 $Comp
-L ArduinoEncoderShield_old-rescue:CONN_2 P4
+L Dorababu:CONN_2 P4
 U 1 1 5C3F0D30
 P 2300 6700
@@
 Spare2
 $Comp
-L ArduinoEncoderShield_old-rescue:R R9
+L Dorababu:R R9
 U 1 1 5C3EFA73
 P 7625 1200
@@
 	7575 1900 7575 1950
 $Comp
-L ArduinoEncoderShield_old-rescue:AGND #PWR04
+L Dorababu:AGND #PWR04
 U 1 1 5C3F0E1A
 P 7625 1450
@@
 $EndComp
 $Comp
-L ArduinoEncoderShield_old-rescue:AGND #PWR03
+L Dorababu:AGND #PWR03
 U 1 1 5C3F0E20
 P 7575 2450
@@
 	6850 3200 7025 3200
 $Comp
-L ArduinoEncoderShield_old-rescue:AGND #PWR06
+L Dorababu:AGND #PWR06
 U 1 1 5C3EFA74
 P 8600 1725
@@
 NoConn ~ 1800 2500
 $Comp
-L ArduinoEncoderShield_old-rescue:ARDUINO_SHIELD SHIELD1
+L DoraBabu:ARDUINO_SHIELD SHIELD1
 U 1 1 5C3EFA63
 P 2750 2800
@@
 	6825 1900 6875 1900
 $Comp
-L ArduinoEncoderShield_old-rescue:AGND #PWR0101
+L Dorababu:AGND #PWR0101
 U 1 1 5D23393F
 P 5050 2725
@@
 $EndComp
 $Comp
-L ArduinoEncoderShield_old-rescue:AGND #PWR0102
+L Dorababu:AGND #PWR0102
 U 1 1 5D239D97
 P 1450 2750

Commit message: Needs to do layout.
Parts:
- CN1: footprint Connector_PinHeader_2.54mm:PinHeader_1x15_P2.54mm_Horizontal -> pinhead-1-1X15/90; symbol Dorababu:HDR-1X15-15-91-? -> DoraBabu:HDR-1X15-15-91-?
- D1: footprint Diode_THT:D_5KP_P12.70mm_Horizontal -> D4; symbol Dorababu:DIODE -> DoraBabu:DIODE
- IC1, IC2, IC3, IC4, IC5: footprint Package_DIP:DIP-6_W7.62mm_Socket -> DIP-6__300_ELL
- J2: footprint (none) -> Connector_PinSocket_2.54mm:PinSocket_1x09_P2.54mm_Horizontal
- P1: footprint Connector_PinHeader_1.27mm:PinHeader_1x06_P1.27mm_Horizontal -> pinhead-1-1X06/90; symbol Dorababu:CONN_6 -> DoraBabu:CONN_6
- P2: footprint Connector_PinHeader_1.27mm:PinHeader_1x06_P1.27mm_Horizontal -> pinhead-1-1X02; symbol Dorababu:CONN_6 -> DoraBabu:CONN_6
- P4: footprint Connector_PinHeader_1.27mm:PinHeader_1x02_P1.27mm_Vertical -> pinhead-1-1X02; symbol Dorababu:CONN_2 -> DoraBabu:CONN_2
- P7: footprint (none) -> pinhead-1-1X05; symbol Dorababu:CONN_2 -> DoraBabu:CONN_2
- P8: footprint Connector_PinHeader_1.27mm:PinHeader_1x08_P1.27mm_Horizontal -> pinhead-1-1X05; symbol Dorababu:CONN_8 -> DoraBabu:CONN_8
- P9: footprint Connector_PinHeader_1.27mm:PinHeader_1x08_P1.27mm_Horizontal -> pinhead-1-1X02/90; symbol Dorababu:CONN_8 -> DoraBabu:CONN_8
- R1, R2: footprint Resistor_SMD:R_0603_1608Metric_Pad1.05x0.95mm_HandSolder -> SM0805; symbol Dorababu:R -> DoraBabu:R
- R10, R11, R12, R4, R5, R6, R7, R8, R9: footprint Resistor_SMD:R_0805_2012Metric_Pad1.15x1.40mm_HandSolder -> SM0805; symbol Dorababu:R -> DoraBabu:R
- R13: symbol Dorababu:R -> DoraBabu:R
- R3: footprint Potentiometer_THT:Potentiometer_Alps_RK09K_Single_Vertical -> SM0805
- SHIELD1: footprint (none) -> Module:Arduino_UNO_R3_WithMountingHoles
- U1: footprint Package_DIP:DIP-16_W7.62mm_Socket -> DIP-16__300_ELL; symbol Dorababu:ULN2003A -> DoraBabu:ULN2003A

Commit message: reassigned PCB components.
Parts:
- CN1: footprint pinhead-1-1X15/90 -> Connector_PinHeader_2.54mm:PinHeader_1x15_P2.54mm_Horizontal; symbol DoraBabu:HDR-1X15-15-91-? -> Schematic-rescue:HDR-1X15-15-91-?-DoraBabu
- D1: footprint D4 -> Diode_THT:D_5KPW_P12.70mm_Horizontal; symbol DoraBabu:DIODE -> Schematic-rescue:DIODE-DoraBabu
- IC1, IC2, IC3, IC4, IC5: footprint DIP-6__300_ELL -> Package_DIP:DIP-6_W7.62mm_Socket
- P1: footprint pinhead-1-1X06/90 -> Connector_PinHeader_2.54mm:PinHeader_1x07_P2.54mm_Horizontal; symbol DoraBabu:CONN_6 -> Schematic-rescue:CONN_6-DoraBabu
- P2: footprint pinhead-1-1X02 -> Connector_PinHeader_2.54mm:PinHeader_1x07_P2.54mm_Horizontal; symbol DoraBabu:CONN_6 -> Schematic-rescue:CONN_6-DoraBabu
- P4: footprint pinhead-1-1X02 -> Connector_PinHeader_2.54mm:PinHeader_1x02_P2.54mm_Horizontal; symbol DoraBabu:CONN_2 -> Schematic-rescue:CONN_2-DoraBabu
- P7: footprint pinhead-1-1X05 -> Connector_PinHeader_2.54mm:PinHeader_1x01_P2.54mm_Vertical; symbol DoraBabu:CONN_2 -> Schematic-rescue:CONN_2-DoraBabu
- P8: footprint pinhead-1-1X05 -> Connector_PinHeader_2.54mm:PinHeader_1x08_P2.54mm_Horizontal; symbol DoraBabu:CONN_8 -> Schematic-rescue:CONN_8-DoraBabu
- P9: footprint pinhead-1-1X02/90 -> Connector_PinHeader_2.54mm:PinHeader_1x08_P2.54mm_Horizontal; symbol DoraBabu:CONN_8 -> Schematic-rescue:CONN_8-DoraBabu
- R1, R10, R11, R12, R2, R4, R5, R6, R7, R8, R9: footprint SM0805 -> Resistor_SMD:R_0603_1608Metric; symbol DoraBabu:R -> Schematic-rescue:R-DoraBabu
- R13: footprint Resistor_SMD:R_0805_2012Metric_Pad1.15x1.40mm_HandSolder -> Resistor_SMD:R_0603_1608Metric; symbol DoraBabu:R -> Schematic-rescue:R-DoraBabu
- R3: value 10k-1M -> 1M; footprint SM0805 -> Potentiometer_THT:Potentiometer_Alps_RK09K_Single_Horizontal
- SHIELD1: symbol DoraBabu:ARDUINO_SHIELD -> Schematic-rescue:ARDUINO_SHIELD-DoraBabu
- U1: footprint DIP-16__300_ELL -> Package_DIP:DIP-16_W7.62mm_Socket; symbol DoraBabu:ULN2003A -> Schematic-rescue:ULN2003A-DoraBabu

Commit message: Added PCB design. Routing to be done.
Parts:
- removed P1, P2: CONN_6, Connector_PinHeader_2.54mm:PinHeader_1x07_P2.54mm_Horizontal, symbol Schematic-rescue:CONN_6-DoraBabu
- removed P4: CONN_2, Connector_PinHeader_2.54mm:PinHeader_1x02_P2.54mm_Horizontal, symbol Schematic-rescue:CONN_2-DoraBabu
- removed P7: CONN_2, Connector_PinHeader_2.54mm:PinHeader_1x01_P2.54mm_Vertical, symbol Schematic-rescue:CONN_2-DoraBabu
- removed P8, P9: CONN_8, Connector_PinHeader_2.54mm:PinHeader_1x08_P2.54mm_Horizontal, symbol Schematic-rescue:CONN_8-DoraBabu
- removed R1, R2: 560E, Resistor_SMD:R_0603_1608Metric, symbol Schematic-rescue:R-DoraBabu
- added J3: RotaryEncoder, Connector_PinSocket_1.27mm:PinSocket_1x04_P1.27mm_Vertical, symbol Connector_Generic:Conn_01x04
- added J4: AnalogIn, Connector_PinSocket_1.27mm:PinSocket_1x06_P1.27mm_Vertical, symbol Connector_Generic:Conn_01x06
- C1: footprint Capacitor_THT:CP_Axial_L11.0mm_D6.0mm_P18.00mm_Horizontal -> Capacitor_THT:C_Disc_D4.7mm_W2.5mm_P5.00mm
- CN1: symbol Schematic-rescue:HDR-1X15-15-91-?-DoraBabu -> Schematic-rescue:HDR-1X15-15-91-?-DoraBabu-Schematic-rescue
- D1: footprint Diode_THT:D_5KPW_P12.70mm_Horizontal -> Diode_THT:D_DO-27_P5.08mm_Vertical_KathodeUp; symbol Schematic-rescue:DIODE-DoraBabu -> Schematic-rescue:DIODE-DoraBabu-Schematic-rescue
- J-InStimInput1: footprint Connector_BarrelJack:BarrelJack_CUI_PJ-036AH-SMT_Horizontal -> Connector_BarrelJack:BarrelJack_Horizontal
- R10, R11, R12, R13, R4, R5, R6, R7, R8, R9: symbol Schematic-rescue:R-DoraBabu -> Schematic-rescue:R-DoraBabu-Schematic-rescue
- SHIELD1: symbol Schematic-rescue:ARDUINO_SHIELD-DoraBabu -> Schematic-rescue:ARDUINO_SHIELD-DoraBabu-Schematic-rescue
- U1: symbol Schematic-rescue:ULN2003A-DoraBabu -> Schematic-rescue:ULN2003A-DoraBabu-Schematic-rescue
Connections:
- net 5V: now also J3.3 (Pin_3)
- net A0: now also J4.1 (Pin_1)
- net A1: now also J4.2 (Pin_2)
- net A2: now also J4.3 (Pin_3)
- net A3: now also J4.4 (Pin_4)
- net A4: now also J4.5 (Pin_5)
- net A5: now also J4.6 (Pin_6)
- net AGND: now also J3.4 (Pin_4)
- net D2: now also J3.1 (Pin_1)
- net D3: now also J3.2 (Pin_2)
- net D0: no longer names the net of SHIELD1.0
- net D1: no longer names the net of SHIELD1.1
- net D10: no longer names the net of SHIELD1.10
- net RST: no longer names the net of SHIELD1.RST
- net Spare1: no longer names the net of CN1.4
- net Spare2: no longer names the net of CN1.3
- no-connect marks 23 -> 26
Other:
- moved on the sheet: J-InStimInput1, J1, J2, JPad1, JPad2
