File: CAD/KiCAD/AnimalBehaviour.sch (KiCad schematic (older format))
At the start: 28 parts, among them CN1 OutputPad, IC1 4N35, IC2 4N35, IC3 4N35, IC4 4N35, IC5 4N35, J1 SSR-ToInput, J2 SSR-ToOutput, J3 RotaryEncoder, J4 AnalogIn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

Commit message: renamed. Project name and sch file name should match. reverted lib change.
Parts:
- CN1: symbol Schematic-rescue:HDR-1X15-15-91-?-DoraBabu-Schematic-rescue -> DoraBabu:HDR-1X15-15-91-?
- D1: symbol Schematic-rescue:DIODE-DoraBabu-Schematic-rescue -> DoraBabu:DIODE
- R10, R11, R12, R13, R4, R5, R6, R7, R8, R9: symbol Schematic-rescue:R-DoraBabu-Schematic-rescue -> DoraBabu:R
- SHIELD1: symbol Schematic-rescue:ARDUINO_SHIELD-DoraBabu-Schematic-rescue -> DoraBabu:ARDUINO_SHIELD
- U1: symbol Schematic-rescue:ULN2003A-DoraBabu-Schematic-rescue -> DoraBabu:ULN2003A
Changed lines of the file:
@@
 EESchema Schematic File Version 4
-LIBS:Schematic-cache
+LIBS:DoraBabu
 EELAYER 29 0
 EELAYER END
@@
 $EndComp
 $Comp
-L Schematic-rescue:ULN2003A-DoraBabu-Schematic-rescue U1
+L DoraBabu:ULN2003A U1
 U 1 1 5C3EFA71
 P 9300 1225
@@
 $EndComp
 $Comp
-L Schematic-rescue:DIODE-DoraBabu-Schematic-rescue D1
+L DoraBabu:DIODE D1
 U 1 1 5C3EFA72
 P 10300 1625
@@
 $EndComp
 $Comp
-L Schematic-rescue:R-DoraBabu-Schematic-rescue R8
+L DoraBabu:R R8
 U 1 1 5C3EFA76
 P 7575 2200
@@
 $EndComp
 $Comp
-L Schematic-rescue:R-DoraBabu-Schematic-rescue R6
+L DoraBabu:R R6
 U 1 1 5C3EFA82
 P 6575 1700
@@
 $EndComp
 $Comp
-L Schematic-rescue:R-DoraBabu-Schematic-rescue R5
+L DoraBabu:R R5
 U 1 1 5C3EFA83
 P 6575 700
@@
 $EndComp
 $Comp
-L Schematic-rescue:R-DoraBabu-Schematic-rescue R10
+L DoraBabu:R R10
 U 1 1 5C3EFA84
 P 7925 5425
@@
 Solenoid2_2
 $Comp
-L Schematic-rescue:HDR-1X15-15-91-?-DoraBabu-Schematic-rescue CN1
+L DoraBabu:HDR-1X15-15-91-? CN1
 U 1 1 5C3EFA8D
 P 1650 5500
@@
 $EndComp
 $Comp
-L Schematic-rescue:R-DoraBabu-Schematic-rescue R12
+L DoraBabu:R R12
 U 1 1 5C3EFA8E
 P 9825 5425
@@
 EX 5 V
 $Comp
-L Schematic-rescue:R-DoraBabu-Schematic-rescue R11
+L DoraBabu:R R11
 U 1 1 5C3F0A84
 P 8875 5975
@@
 	8875 5725 8875 5675
 $Comp
-L Schematic-rescue:AGND-DoraBabu-Schematic-rescue #PWR05
+L DoraBabu:AGND #PWR05
 U 1 1 5C3F0AE2
 P 8875 6325
@@
 DGND
 $Comp
-L Schematic-rescue:R-DoraBabu-Schematic-rescue R13
+L DoraBabu:R R13
 U 1 1 5C3F0BA2
 P 10775 5975
@@
 $EndComp
 $Comp
-L Schematic-rescue:AGND-DoraBabu-Schematic-rescue #PWR07
+L DoraBabu:AGND #PWR07
 U 1 1 5C3F0BA8
 P 10775 6325
@@
 AGND
 $Comp
-L Schematic-rescue:AGND-DoraBabu-Schematic-rescue #PWR02
+L DoraBabu:AGND #PWR02
 U 1 1 5C3F0CE1
 P 6975 6225
@@
 AGND
 $Comp
-L Schematic-rescue:R-DoraBabu-Schematic-rescue R9
+L DoraBabu:R R9
 U 1 1 5C3EFA73
 P 7625 1200
@@
 	7575 1900 7575 1950
 $Comp
-L Schematic-rescue:AGND-DoraBabu-Schematic-rescue #PWR04
+L DoraBabu:AGND #PWR04
 U 1 1 5C3F0E1A
 P 7625 1450
@@
 $EndComp
 $Comp
-L Schematic-rescue:AGND-DoraBabu-Schematic-rescue #PWR03
+L DoraBabu:AGND #PWR03
 U 1 1 5C3F0E20
 P 7575 2450
@@
 	6750 3650 6925 3650
 $Comp
-L Schematic-rescue:AGND-DoraBabu-Schematic-rescue #PWR06
+L DoraBabu:AGND #PWR06
 U 1 1 5C3EFA74
 P 8600 1725
@@
 	6825 1900 6875 1900
 $Comp
-L Schematic-rescue:AGND-DoraBabu-Schematic-rescue #PWR0101
+L DoraBabu:AGND #PWR0101
 U 1 1 5D23393F
 P 5050 2725
@@
 NoConn ~ 1800 2900
 $Comp
-L Schematic-rescue:R-DoraBabu-Schematic-rescue R4
+L DoraBabu:R R4
 U 1 1 5C3EFA94
 P 5975 5425
@@
 $EndComp
 $Comp
-L Schematic-rescue:R-DoraBabu-Schematic-rescue R7
+L DoraBabu:R R7
 U 1 1 5C3EFA96
 P 6975 5925
@@
 	1800 2700 1625 2700
 $Comp
-L Schematic-rescue:AGND-DoraBabu-Schematic-rescue #PWR0102
+L DoraBabu:AGND #PWR0102
 U 1 1 5D239D97
 P 1450 2750
@@
 $EndComp
 $Comp
-L Schematic-rescue:ARDUINO_SHIELD-DoraBabu-Schematic-rescue SHIELD1
+L DoraBabu:ARDUINO_SHIELD SHIELD1
 U 1 1 5C3EFA63
 P 2750 2800
@@
 $EndComp
 $Comp
-L Schematic-rescue:AGND-DoraBabu-Schematic-rescue #PWR01
+L DoraBabu:AGND #PWR01
 U 1 1 5D23D211
 P 6650 3300

Commit message: recued symbols.
Parts:
- CN1: symbol DoraBabu:HDR-1X15-15-91-? -> DoraBabu:ArduinoEncoderShield_old-rescue_HDR-1X15-15-91-?
- D1: symbol DoraBabu:DIODE -> DoraBabu:ArduinoEncoderShield_old-rescue_DIODE
- R10, R11, R12, R13, R4, R5, R6, R7, R8, R9: symbol DoraBabu:R -> DoraBabu:ArduinoEncoderShield_old-rescue_R
- SHIELD1: symbol DoraBabu:ARDUINO_SHIELD -> DoraBabu:ArduinoEncoderShield_old-rescue_ARDUINO_SHIELD
- U1: symbol DoraBabu:ULN2003A -> DoraBabu:ArduinoEncoderShield_old-rescue_ULN2003A
Changed lines of the file:
@@
 EESchema Schematic File Version 4
-LIBS:DoraBabu
 EELAYER 29 0
 EELAYER END
@@
 $EndComp
 $Comp
-L DoraBabu:ULN2003A U1
+L DoraBabu:ArduinoEncoderShield_old-rescue_ULN2003A U1
 U 1 1 5C3EFA71
 P 9300 1225
@@
 $EndComp
 $Comp
-L DoraBabu:DIODE D1
+L DoraBabu:ArduinoEncoderShield_old-rescue_DIODE D1
 U 1 1 5C3EFA72
 P 10300 1625
@@
 $EndComp
 $Comp
-L DoraBabu:R R8
+L DoraBabu:ArduinoEncoderShield_old-rescue_R R8
 U 1 1 5C3EFA76
 P 7575 2200
@@
 $EndComp
 $Comp
-L DoraBabu:R R6
+L DoraBabu:ArduinoEncoderShield_old-rescue_R R6
 U 1 1 5C3EFA82
 P 6575 1700
@@
 $EndComp
 $Comp
-L DoraBabu:R R5
+L DoraBabu:ArduinoEncoderShield_old-rescue_R R5
 U 1 1 5C3EFA83
 P 6575 700
@@
 $EndComp
 $Comp
-L DoraBabu:R R10
+L DoraBabu:ArduinoEncoderShield_old-rescue_R R10
 U 1 1 5C3EFA84
 P 7925 5425
@@
 Solenoid2_2
 $Comp
-L DoraBabu:HDR-1X15-15-91-? CN1
+L DoraBabu:ArduinoEncoderShield_old-rescue_HDR-1X15-15-91-? CN1
 U 1 1 5C3EFA8D
 P 1650 5500
@@
 $EndComp
 $Comp
-L DoraBabu:R R12
+L DoraBabu:ArduinoEncoderShield_old-rescue_R R12
 U 1 1 5C3EFA8E
 P 9825 5425
@@
 EX 5 V
 $Comp
-L DoraBabu:R R11
+L DoraBabu:ArduinoEncoderShield_old-rescue_R R11
 U 1 1 5C3F0A84
 P 8875 5975
@@
 	8875 5725 8875 5675
 $Comp
-L DoraBabu:AGND #PWR05
+L power:GNDA #PWR05
 U 1 1 5C3F0AE2
 P 8875 6325
@@
 DGND
 $Comp
-L DoraBabu:R R13
+L DoraBabu:ArduinoEncoderShield_old-rescue_R R13
 U 1 1 5C3F0BA2
 P 10775 5975
@@
 $EndComp
 $Comp
-L DoraBabu:AGND #PWR07
+L power:GNDA #PWR07
 U 1 1 5C3F0BA8
 P 10775 6325
@@
 AGND
 $Comp
-L DoraBabu:AGND #PWR02
+L power:GNDA #PWR02
 U 1 1 5C3F0CE1
 P 6975 6225
@@
 AGND
 $Comp
-L DoraBabu:R R9
+L DoraBabu:ArduinoEncoderShield_old-rescue_R R9
 U 1 1 5C3EFA73
 P 7625 1200
@@
 	7575 1900 7575 1950
 $Comp
-L DoraBabu:AGND #PWR04
+L power:GNDA #PWR04
 U 1 1 5C3F0E1A
 P 7625 1450
@@
 $EndComp
 $Comp
-L DoraBabu:AGND #PWR03
+L power:GNDA #PWR03
 U 1 1 5C3F0E20
 P 7575 2450
@@
 	6750 3650 6925 3650
 $Comp
-L DoraBabu:AGND #PWR06
+L power:GNDA #PWR06
 U 1 1 5C3EFA74
 P 8600 1725
@@
 	6825 1900 6875 1900
 $Comp
-L DoraBabu:AGND #PWR0101
+L power:GNDA #PWR0101
 U 1 1 5D23393F
 P 5050 2725
@@
 NoConn ~ 1800 2900
 $Comp
-L DoraBabu:R R4
+L DoraBabu:ArduinoEncoderShield_old-rescue_R R4
 U 1 1 5C3EFA94
 P 5975 5425
@@
 $EndComp
 $Comp
-L DoraBabu:R R7
+L DoraBabu:ArduinoEncoderShield_old-rescue_R R7
 U 1 1 5C3EFA96
 P 6975 5925
@@
 	1800 2700 1625 2700
 $Comp
-L DoraBabu:AGND #PWR0102
+L power:GNDA #PWR0102
 U 1 1 5D239D97
 P 1450 2750
@@
 $EndComp
 $Comp
-L DoraBabu:ARDUINO_SHIELD SHIELD1
+L DoraBabu:ArduinoEncoderShield_old-rescue_ARDUINO_SHIELD SHIELD1
 U 1 1 5C3EFA63
 P 2750 2800
@@
 $EndComp
 $Comp
-L DoraBabu:AGND #PWR01
+L power:GNDA #PWR01
 U 1 1 5D23D211
 P 6650 3300
