File: CAD/KiCAD/AnimalBehaviour.sch (KiCad schematic (older format))
At the start: 28 parts, among them J1 Conn_01x06_Male, J10 Conn_01x02_Male, J11 Conn_01x03_Male, J12 Conn_01x02_Male, J2 Conn_01x02_Male, J3 Conn_01x04_Male, J4 Conn_01x08_Male, J5 Conn_01x02_Male, J6 Conn_01x02_Male, J7 Jack-DC, J8 Conn_01x02_Male, J9 Conn_Coaxial, P1 CONN_6, P2 CONN_6, P3 CONN_8, P4 CONN_8, Q1 IRF540N, U1 4N35

Commit message: Added today's snapshot.
Parts:
- D1: symbol ArduinoEncoderShield_anzal-rescue:DIODE -> AnimalBehaviour-rescue:DIODE-ArduinoEncoderShield_anzal-rescue
- P1, P2: symbol ArduinoEncoderShield_anzal-rescue:CONN_6 -> AnimalBehaviour-rescue:CONN_6-ArduinoEncoderShield_anzal-rescue
- P3, P4: symbol ArduinoEncoderShield_anzal-rescue:CONN_8 -> AnimalBehaviour-rescue:CONN_8-ArduinoEncoderShield_anzal-rescue
- R1, R2, R3, R4, R5, R6: symbol ArduinoEncoderShield_anzal-rescue:R -> AnimalBehaviour-rescue:R-ArduinoEncoderShield_anzal-rescue
- SHIELD1: symbol ArduinoEncoderShield_anzal-rescue:ARDUINO_SHIELD -> AnimalBehaviour-rescue:ARDUINO_SHIELD-ArduinoEncoderShield_anzal-rescue
Changed lines of the file:
@@
 EESchema Schematic File Version 4
-LIBS:ArduinoEncoderShield_anzal-cache
+LIBS:AnimalBehaviour-cache
 EELAYER 29 0
 EELAYER END
@@
 $EndDescr
 $Comp
-L ArduinoEncoderShield_anzal-rescue:ARDUINO_SHIELD SHIELD1
+L AnimalBehaviour-rescue:ARDUINO_SHIELD-ArduinoEncoderShield_anzal-rescue SHIELD1
 U 1 1 5C3EFA63
 P 6450 2300
@@
 $EndComp
 $Comp
-L ArduinoEncoderShield_anzal-rescue:CONN_8 P4
+L AnimalBehaviour-rescue:CONN_8-ArduinoEncoderShield_anzal-rescue P4
 U 1 1 5C3EFA87
 P 8450 2750
@@
 $EndComp
 $Comp
-L ArduinoEncoderShield_anzal-rescue:CONN_6 P2
+L AnimalBehaviour-rescue:CONN_6-ArduinoEncoderShield_anzal-rescue P2
 U 1 1 5C3EFA88
 P 4400 2850
@@
 $EndComp
 $Comp
-L ArduinoEncoderShield_anzal-rescue:R R1
+L AnimalBehaviour-rescue:R-ArduinoEncoderShield_anzal-rescue R1
 U 1 1 5C3EFA9A
 P 2100 1850
@@
 AREF
 $Comp
-L ArduinoEncoderShield_anzal-rescue:CONN_8 P3
+L AnimalBehaviour-rescue:CONN_8-ArduinoEncoderShield_anzal-rescue P3
 U 1 1 5C3EFD0C
 P 8450 1850
@@
 AREF
 $Comp
-L ArduinoEncoderShield_anzal-rescue:CONN_6 P1
+L AnimalBehaviour-rescue:CONN_6-ArduinoEncoderShield_anzal-rescue P1
 U 1 1 5C3F096C
 P 4400 2150
@@
 	1850 1950 1800 1950
 $Comp
-L ArduinoEncoderShield_anzal-rescue:R R2
+L AnimalBehaviour-rescue:R-ArduinoEncoderShield_anzal-rescue R2
 U 1 1 5C3EFA99
 P 2100 1950
@@
 $EndComp
 $Comp
-L ArduinoEncoderShield_anzal-rescue:R R5
+L AnimalBehaviour-rescue:R-ArduinoEncoderShield_anzal-rescue R5
 U 1 1 5D221F97
 P 8300 4150
@@
 DGND
 $Comp
-L ArduinoEncoderShield_anzal-rescue:R R6
+L AnimalBehaviour-rescue:R-ArduinoEncoderShield_anzal-rescue R6
 U 1 1 5D222B56
 P 9200 4650
@@
 	9950 4050 9950 4150
 $Comp
-L ArduinoEncoderShield_anzal-rescue:DIODE D1
+L AnimalBehaviour-rescue:DIODE-ArduinoEncoderShield_anzal-rescue D1
 U 1 1 5D22A71C
 P 9700 3950
@@
 $EndComp
 $Comp
-L ArduinoEncoderShield_anzal-rescue:R R4
+L AnimalBehaviour-rescue:R-ArduinoEncoderShield_anzal-rescue R4
 U 1 1 5D261F4B
 P 6900 5250
@@
 Extra pin for new arduino version\n
 $Comp
-L ArduinoEncoderShield_anzal-rescue:R R3
+L AnimalBehaviour-rescue:R-ArduinoEncoderShield_anzal-rescue R3
 U 1 1 5D21C427
 P 5500 6700

Commit message: Added new schematics, aduino footprints etc.
Parts:
- removed R1: 560E, Resistors_ThroughHole:R_Axial_DIN0309_L9.0mm_D3.2mm_P12.70mm_Horizontal, symbol AnimalBehaviour-rescue:R-ArduinoEncoderShield_anzal-rescue
- removed R2: 560E, Resistors_ThroughHole:R_Axial_DIN0411_L9.9mm_D3.6mm_P12.70mm_Horizontal, symbol AnimalBehaviour-rescue:R-ArduinoEncoderShield_anzal-rescue
- removed SHIELD1: ARDUINO_SHIELD, arduino_shields:ARDUINO_SHIELD_040pins, symbol AnimalBehaviour-rescue:ARDUINO_SHIELD-ArduinoEncoderShield_anzal-rescue
- added XA1: Arduino_Uno_Shield, Arduino:Arduino_Uno_Shield, symbol arduino:Arduino_Uno_Shield
- C1: footprint Capacitors_ThroughHole:CP_Radial_D10.0mm_P5.00mm -> Capacitor_THT:CP_Radial_D5.0mm_P2.00mm
- D1: footprint Diodes_ThroughHole:D_5KP_P12.70mm_Horizontal -> Diode_THT:D_DO-15_P12.70mm_Horizontal; symbol AnimalBehaviour-rescue:DIODE-ArduinoEncoderShield_anzal-rescue -> AnimalBehaviour-rescue:DIODE-ArduinoEncoderShield_anzal-rescue-AnimalBehaviour-rescue
- J1: footprint Connectors_Molex:Molex_NanoFit_1x06x2.50mm_Straight -> Connector_Molex:Molex_KK-254_AE-6410-06A_1x06_P2.54mm_Vertical
- J10, J12, J2, J5, J6, J8: footprint Connectors_Molex:Molex_NanoFit_1x02x2.50mm_Straight -> Connector_Molex:Molex_KK-254_AE-6410-02A_1x02_P2.54mm_Vertical
- J11: footprint Connectors_Molex:Molex_NanoFit_1x03x2.50mm_Straight -> Connector_Molex:Molex_KK-254_AE-6410-03A_1x03_P2.54mm_Vertical
- J3: footprint Connectors_Molex:Molex_NanoFit_1x04x2.50mm_Straight -> Connector_Molex:Molex_KK-254_AE-6410-04A_1x04_P2.54mm_Vertical
- J4: footprint Connectors_Molex:Molex_NanoFit_1x08x2.50mm_Straight -> Connector_Molex:Molex_KK-254_AE-6410-08A_1x08_P2.54mm_Vertical
- J7: footprint Connect:Barrel_Jack_CUI_PJ-102AH -> Connector_BarrelJack:BarrelJack_CUI_PJ-063AH_Horizontal
- J9: footprint w_conn_rf:bnc_90_1-1337543-0 -> Connector_Coaxial:BNC_TEConnectivity_1478204_Vertical
- P1, P2: footprint Connectors_Molex:Molex_NanoFit_1x06x2.50mm_Straight -> Connector_Molex:Molex_KK-254_AE-6410-06A_1x06_P2.54mm_Vertical; symbol AnimalBehaviour-rescue:CONN_6-ArduinoEncoderShield_anzal-rescue -> Connector_Generic:Conn_01x06
- P3, P4: footprint Connectors_Molex:Molex_NanoFit_1x08x2.50mm_Straight -> Connector_Molex:Molex_KK-254_AE-6410-08A_1x08_P2.54mm_Vertical; symbol AnimalBehaviour-rescue:CONN_8-ArduinoEncoderShield_anzal-rescue -> Connector_Generic:Conn_01x08
- Q1: footprint TO_SOT_Packages_THT:TO-220-3_Vertical -> Package_TO_SOT_THT:TO-220-3_Horizontal_TabDown
- R1: renamed from R3; footprint Resistors_ThroughHole:R_Axial_DIN0411_L9.9mm_D3.6mm_P12.70mm_Horizontal -> Resistor_THT:R_Axial_DIN0414_L11.9mm_D4.5mm_P25.40mm_Horizontal; symbol AnimalBehaviour-rescue:R-ArduinoEncoderShield_anzal-rescue -> AnimalBehaviour-rescue:R-ArduinoEncoderShield_anzal-rescue-AnimalBehaviour-rescue
- R2: renamed from R4; footprint Resistors_ThroughHole:R_Axial_DIN0411_L9.9mm_D3.6mm_P12.70mm_Horizontal -> Resistor_THT:R_Axial_DIN0414_L11.9mm_D4.5mm_P25.40mm_Horizontal; symbol AnimalBehaviour-rescue:R-ArduinoEncoderShield_anzal-rescue -> AnimalBehaviour-rescue:R-ArduinoEncoderShield_anzal-rescue-AnimalBehaviour-rescue
- R3: renamed from R5; footprint Resistors_ThroughHole:R_Axial_DIN0411_L9.9mm_D3.6mm_P12.70mm_Horizontal -> Resistor_THT:R_Axial_DIN0414_L11.9mm_D4.5mm_P25.40mm_Horizontal; symbol AnimalBehaviour-rescue:R-ArduinoEncoderShield_anzal-rescue -> AnimalBehaviour-rescue:R-ArduinoEncoderShield_anzal-rescue-AnimalBehaviour-rescue
- R4: renamed from R6; footprint Resistors_ThroughHole:R_Axial_DIN0411_L9.9mm_D3.6mm_P12.70mm_Horizontal -> Resistor_THT:R_Axial_DIN0414_L11.9mm_D4.5mm_P25.40mm_Horizontal; symbol AnimalBehaviour-rescue:R-ArduinoEncoderShield_anzal-rescue -> AnimalBehaviour-rescue:R-ArduinoEncoderShield_anzal-rescue-AnimalBehaviour-rescue
- RV1: footprint Connect:PINHEAD1-3 -> Potentiometer_THT:Potentiometer_ACP_CA14V-15_Vertical_Hole
- U1: footprint Housings_DIP:DIP-6_W7.62mm_Socket_LongPads -> Package_DIP:DIP-6_W7.62mm_Socket
Connections:
- net labels added: GNDD
- net labels removed: D0, D1, GND
- wire segments 55 -> 53
- no-connect marks 0 -> 9

Commit message: ERC passed with assign PWR_FLAGS. See this for more information https://forum.kicad.info/t/errtype-3-pin-connected-to-some-others-pins-but-no-pin-to-drive-it/10946/4
Parts:
- D1: symbol AnimalBehaviour-rescue:DIODE-ArduinoEncoderShield_anzal-rescue-AnimalBehaviour-rescue -> Device:D
- R1, R2, R3, R4: symbol AnimalBehaviour-rescue:R-ArduinoEncoderShield_anzal-rescue-AnimalBehaviour-rescue -> Device:R
Connections:
- net GNDD: now also XA1.GND2 (GND), XA1.GND3 (GND)
- no-connect marks 9 -> 15
Changed lines of the file:
@@
 Text GLabel 4750 1900 2    60   Input ~ 0
 RST
-Text GLabel 4750 2000 2    60   Input ~ 0
-3V3
-Text GLabel 4750 2100 2    60   Input ~ 0
-5V
 Text GLabel 4750 2200 2    60   Input ~ 0
 DGND
 Text GLabel 4750 2300 2    60   Input ~ 0
 DGND
-Text GLabel 4750 2400 2    60   Input ~ 0
+Text GLabel 5225 2400 2    60   Input ~ 0
 V_IN
 Text GLabel 8550 3450 2    60   Input ~ 0
 RST
-Text GLabel 5950 3350 0    60   Input ~ 0
-3V3
-Text GLabel 5950 3450 0    60   Input ~ 0
-5V
-Text GLabel 5950 3050 0    60   Input ~ 0
-DGND
-Text GLabel 5950 3550 0    60   Input ~ 0
-V_IN
 Text GLabel 4750 2600 2    60   Input ~ 0
 A0
@@
 Wire Wire Line
 	1800 2050 2400 2050
-Wire Wire Line
-	1800 2150 2250 2150
 Text GLabel 1950 5100 2    60   Input ~ 0
 D6
@@
 Text Notes 1850 4250 0    50   ~ 10
 SSR Relay\n
-Wire Wire Line
-	2250 2200 2250 2150
-Connection ~ 2250 2150
-Wire Wire Line
-	2250 2150 2400 2150
 Text Notes 5650 6300 0    50   ~ 10
 LED\n
@@
 	1    0    0    -1
 $EndComp
-$Comp
-L AnimalBehaviour-rescue:R-ArduinoEncoderShield_anzal-rescue-AnimalBehaviour-rescue R3
-U 1 1 5D221F97
-P 8300 4150
-F 0 "R3" V 8115 4150 40  0000 C CNN
-F 1 "470E" V 8191 4150 40  0000 C CNN
-F 2 "Resistor_THT:R_Axial_DIN0414_L11.9mm_D4.5mm_P25.40mm_Horizontal" V 8230 4150 30  0001 C CNN
-F 3 "" H 8300 4150 30  0000 C CNN
-	1    8300 4150
-	0    1    1    0
-$EndComp
 Text GLabel 8050 4150 0    60   Input ~ 0
 D11
@@
 DGND
 $Comp
-L AnimalBehaviour-rescue:R-ArduinoEncoderShield_anzal-rescue-AnimalBehaviour-rescue R4
+L Device:R R4
 U 1 1 5D222B56
 P 9200 4650
@@
 Wire Wire Line
 	9150 4350 9200 4350
-Wire Wire Line
-	9200 4350 9200 4400
 Text GLabel 9200 5000 0    60   Input ~ 0
 AGND
@@
 	9950 4950 9200 4950
 Connection ~ 9200 4950
-Wire Wire Line
-	9200 4950 9200 4900
 $Comp
 L Connector:Conn_01x02_Male J12
@@
 	9950 4050 9950 4150
 $Comp
-L AnimalBehaviour-rescue:DIODE-ArduinoEncoderShield_anzal-rescue-AnimalBehaviour-rescue D1
+L Device:D D1
 U 1 1 5D22A71C
 P 9700 3950
@@
 $EndComp
 $Comp
-L AnimalBehaviour-rescue:R-ArduinoEncoderShield_anzal-rescue-AnimalBehaviour-rescue R2
+L Device:R R2
 U 1 1 5D261F4B
 P 6900 5250
@@
 A0
 Wire Wire Line
-	6900 5500 7250 5500
-Wire Wire Line
 	7250 5500 7250 5450
 Wire Wire Line
@@
 Text GLabel 6750 5500 0    60   Input ~ 0
 DGND
-Wire Wire Line
-	6750 5500 6900 5500
-Connection ~ 6900 5500
 Wire Wire Line
 	6900 5000 7050 5000
@@
 Text GLabel 2000 3600 2    60   Input ~ 0
 Vcc
-Text GLabel 1750 3600 0    60   Input ~ 0
-5V
-Wire Wire Line
-	1750 3600 2000 3600
 Text GLabel 5250 6700 0    60   Input ~ 0
 D9
 Text Notes 4600 800  0    60   ~ 0
 Extra pin for new arduino version\n
-$Comp
-L AnimalBehaviour-rescue:R-ArduinoEncoderShield_anzal-rescue-AnimalBehaviour-rescue R1
-U 1 1 5D21C427
-P 5500 6700
-F 0 "R1" V 5315 6700 40  0000 C CNN
-F 1 "470E" V 5391 6700 40  0000 C CNN
-F 2 "Resistor_THT:R_Axial_DIN0414_L11.9mm_D4.5mm_P25.40mm_Horizontal" V 5430 6700 30  0001 C CNN
-F 3 "" H 5500 6700 30  0000 C CNN
-	1    5500 6700
-	0    1    1    0
-$EndComp
 Text GLabel 5400 6800 0    60   Input ~ 0
 DGND
@@
 	5400 6800 5850 6800
 Wire Wire Line
-	5850 6700 5750 6700
-Wire Wire Line
 	1800 1850 2400 1850
 Wire Wire Line
 	1800 1950 2400 1950
 NoConn ~ 6900 4900
-$Comp
-L power:GNDD #PWR02
-U 1 1 5D2143A2
-P 2250 2200
-F 0 "#PWR02" H 2250 1950 50  0001 C CNN
-F 1 "GNDD" H 2254 2045 50  0000 C CNN
-F 2 "" H 2250 2200 50  0001 C CNN
-F 3 "" H 2250 2200 50  0001 C CNN
-	1    2250 2200
-	1    0    0    -1
-$EndComp
-$Comp
-L power:GNDD #PWR01
-U 1 1 5D2152C0
-P 1900 4750
-F 0 "#PWR01" H 1900 4500 50  0001 C CNN
-F 1 "GNDD" V 1904 4640 50  0000 R CNN
-F 2 "" H 1900 4750 50  0001 C CNN
-F 3 "" H 1900 4750 50  0001 C CNN
-	1    1900 4750
-	0    -1   -1   0
-$EndComp
-NoConn ~ 5950 3150
 Text GLabel 5950 2750 0    60   Input ~ 0
 AREF
@@
 NoConn ~ 5950 1750
 NoConn ~ 5950 1850
+Wire Wire Line
+	6750 5500 6900 5500
+Wire Wire Line
+	6900 5000 6900 5100
+Wire Wire Line
+	6900 5400 6900 5500
+Connection ~ 6900 5500
+Wire Wire Line
+	6900 5500 7250 5500
+Wire Wire Line
+	9200 4800 9200 4950
+Wire Wire Line
+	9200 4350 9200 4500
+Wire Wire Line
+	9700 3750 9700 3800
+Wire Wire Line
+	9700 4100 9700 4150
+Text GLabel 1900 4750 2    60   Input ~ 0
+DGND
+$Comp
+L Device:R R3
+U 1 1 5D221F97
+P 8300 4150
+F 0 "R3" V 8115 4150 40  0000 C CNN
+F 1 "470E" V 8191 4150 40  0000 C CNN
+F 2 "Resistor_THT:R_Axial_DIN0414_L11.9mm_D4.5mm_P25.40mm_Horizontal" V 8230 4150 30  0001 C CNN
+F 3 "" H 8300 4150 30  0000 C CNN
+	1    8300 4150
+	0    1    1    0
+$EndComp
+Wire Wire Line
+	8050 4150 8150 4150
+Wire Wire Line
+	8450 4150 8550 4150
+$Comp
+L Device:R R1
+U 1 1 5D21C427
+P 5500 6700
+F 0 "R1" V 5315 6700 40  0000 C CNN
+F 1 "470E" V 5391 6700 40  0000 C CNN
+F 2 "Resistor_THT:R_Axial_DIN0414_L11.9mm_D4.5mm_P25.40mm_Horizontal" V 5430 6700 30  0001 C CNN
+F 3 "" H 5500 6700 30  0000 C CNN
+	1    5500 6700
+	0    1    1    0
+$EndComp
+Wire Wire Line
+	5650 6700 5850 6700
+Wire Wire Line
+	5350 6700 5250 6700
+Text GLabel 2000 3775 2    60   Input ~ 0
+DGND
+Wire Wire Line
+	1750 3775 2000 3775
+Text GLabel 5950 3550 0    60   Input ~ 0
+V_IN
+$Comp
+L power:GNDD #PWR0101
+U 1 1 5D21B10A
+P 1750 3775
+F 0 "#PWR0101" H 1750 3525 50  0001 C CNN
+F 1 "GNDD" V 1754 3665 50  0000 R CNN
+F 2 "" H 1750 3775 50  0001 C CNN
+F 3 "" H 1750 3775 50  0001 C CNN
+	1    1750 3775
+	0    1    1    0
+$EndComp
+Wire Wire Line
+	1750 3600 2000 3600
+Text GLabel 1750 3600 0    60   Input ~ 0
+5V
+Text GLabel 5950 3250 0    60   Input ~ 0
+DGND
+Text GLabel 5950 3150 0    60   Input ~ 0
+DGND
+Text GLabel 5950 3050 0    60   Input ~ 0
+DGND
+Text GLabel 5950 3450 0    60   Input ~ 0
+5V
+Text GLabel 5950 3350 0    60   Input ~ 0
+3V3
+Text GLabel 5225 2000 2    60   Input ~ 0
+3V3
+Text GLabel 5225 2100 2    60   Input ~ 0
+5V
+NoConn ~ 8550 2750
+NoConn ~ 8550 2850
+NoConn ~ 8550 2950
+NoConn ~ 8550 3050
+NoConn ~ 8550 3150
+NoConn ~ 8550 3250
+NoConn ~ 8550 3550
+$Comp
+L power:PWR_FLAG #FLG0101
+U 1 1 5D249963
+P 5075 1925
+F 0 "#FLG0101" H 5075 2000 50  0001 C CNN
+F 1 "PWR_FLAG" H 5075 2098 50  0000 C CNN
+F 2 "" H 5075 1925 50  0001 C CNN
+F 3 "~" H 5075 1925 50  0001 C CNN
+	1    5075 1925
+	1    0    0    -1
+$EndComp
+Wire Wire Line
+	4750 2000 5075 2000
+Wire Wire Line
+	5075 1925 5075 2000
+Connection ~ 5075 2000
+Wire Wire Line
+	5075 2000 5225 2000
+Wire Wire Line
+	1800 2150 2075 2150
+$Comp
+L power:PWR_FLAG #FLG0102
+U 1 1 5D25020E
+P 2075 2200
+F 0 "#FLG0102" H 2075 2275 50  0001 C CNN
+F 1 "PWR_FLAG" H 2075 2373 50  0000 C CNN
+F 2 "" H 2075 2200 50  0001 C CNN
+F 3 "~" H 2075 2200 50  0001 C CNN
+	1    2075 2200
+	-1   0    0    1
+$EndComp
+Wire Wire Line
+	2075 2200 2075 2150
+Connection ~ 2075 2150
+Wire Wire Line
+	2075 2150 2400 2150
+$Comp
+L power:PWR_FLAG #FLG0103
+U 1 1 5D2522BA
+P 5150 2375
+F 0 "#FLG0103" H 5150 2450 50  0001 C CNN
+F 1 "PWR_FLAG" H 5150 2548 50  0000 C CNN
+F 2 "" H 5150 2375 50  0001 C CNN
+F 3 "~" H 5150 2375 50  0001 C CNN
+	1    5150 2375
+	1    0    0    -1
+$EndComp
+Wire Wire Line
+	4750 2400 5150 2400
+Wire Wire Line
+	5150 2375 5150 2400
+Connection ~ 5150 2400
+Wire Wire Line
+	5150 2400 5225 2400
+$Comp
+L power:PWR_FLAG #FLG0104
+U 1 1 5D25582A
+P 5125 2100
+F 0 "#FLG0104" H 5125 2175 50  0001 C CNN
+F 1 "PWR_FLAG" H 5125 2273 50  0000 C CNN
+F 2 "" H 5125 2100 50  0001 C CNN
+F 3 "~" H 5125 2100 50  0001 C CNN
+	1    5125 2100
+	1    0    0    -1
+$EndComp
+Wire Wire Line
+	4750 2100 5125 2100
+Connection ~ 5125 2100
+Wire Wire Line
+	5125 2100 5225 2100
 $EndSCHEMATC

Commit message: v2019.07.06.alpha1
Parts:
- removed J1: Conn_01x06_Male, Connector_Molex:Molex_KK-254_AE-6410-06A_1x06_P2.54mm_Vertical, symbol Connector:Conn_01x06_Male
- removed J2, J6: Conn_01x02_Male, Connector_Molex:Molex_KK-254_AE-6410-02A_1x02_P2.54mm_Vertical, symbol Connector:Conn_01x02_Male
- removed J3: Conn_01x04_Male, Connector_Molex:Molex_KK-254_AE-6410-04A_1x04_P2.54mm_Vertical, symbol Connector:Conn_01x04_Male
- removed P1, P2: CONN_6, Connector_Molex:Molex_KK-254_AE-6410-06A_1x06_P2.54mm_Vertical, symbol Connector_Generic:Conn_01x06
- removed P3, P4: CONN_8, Connector_Molex:Molex_KK-254_AE-6410-08A_1x08_P2.54mm_Vertical, symbol Connector_Generic:Conn_01x08
- added Assr4ch1: PCB_SSR_4Ch_LLT, SSR4Channel:4ChannelSSR, symbol AnimalBehaviour-rescue:PCB_SSR_4Ch_LLT-BhallaLabComponents
- added J1: SSR_INPUT, Connector_Molex:Molex_KK-254_AE-6410-04A_1x04_P2.54mm_Vertical, symbol Connector_Generic:Conn_01x04
- added J10: Cam, BhallaLab:Connector_Mini-DIN_Female_6Pin_2rows, symbol Connector:DIN-6
- added J11: Imaging, BhallaLab:Connector_Mini-DIN_Female_6Pin_2rows, symbol Connector:DIN-6
- added J7: AudioJack2, Connector_Audio:Jack_3.5mm_CUI_SJ-3523-SMT_Horizontal, symbol Connector:AudioJack2
- added RotaryEncoder1: Orange Optical RotaryEncoder, Connector_Molex:Molex_KK-254_AE-6410-04A_1x04_P2.54mm_Vertical, symbol BhallaLabComponents:OrangeOpticalRotaryEncoder
- added ShockPad1: ShockPad, TerminalBlock:TerminalBlock_Altech_AK300-2_P5.00mm, symbol BhallaLabComponents:PCB-ShockPad
- J2: renamed from J4; value Conn_01x08_Male -> SSR OUT; symbol Connector:Conn_01x08_Male -> Connector_Generic:Conn_01x08
- J3: renamed from J7; value Jack-DC -> StimCurrentInject
- J4: renamed from J9; value Conn_Coaxial -> StimIsoIN
- J5: value Conn_01x02_Male -> ImagingTrig
- J6: renamed from J8; value Conn_01x02_Male -> CAM
- J9: renamed from J10; value Conn_01x02_Male -> LED
- RV1: footprint Potentiometer_THT:Potentiometer_ACP_CA14V-15_Vertical_Hole -> Potentiometer_THT:Potentiometer_Alps_RK09L_Single_Vertical
- renumbered J11 to J8, R2 to R1, R3 to R2, R4 to R3, R1 to R4
Connections:
- net 5V: now also Assr4ch1.DC+, J1.1 (Pin_1), RotaryEncoder1.3 (VCC)
- net GNDD: now also Assr4ch1.DC-, J1.2 (Pin_2), J10.6, J11.6, RotaryEncoder1.4 (GND); no longer XA1.GND2 (GND), XA1.GND3 (GND)
- net OUT+: now also J2.4 (Pin_4), Assr4ch1.A3; no longer J2.5 (Pin_5)
- net OUT-: now also J2.2 (Pin_2), Assr4ch1.A4; no longer J2.7 (Pin_7)
- net PAD+: now also J2.3 (Pin_3), J2.7 (Pin_7), Assr4ch1.B1, Assr4ch1.B3 (A3), ShockPad1.0 (PAD+); no longer J2.2 (Pin_2), J2.6 (Pin_6)
- net PAD-: now also J2.1 (Pin_1), J2.5 (Pin_5), Assr4ch1.B2, Assr4ch1.B4, ShockPad1.1 (PAD-); no longer J2.4 (Pin_4), J2.8 (Pin_8)
- net 3V3: no longer names the net of XA1.3V3 (3.3V)
- net A0 renamed ShockRead
- net ShockRead: now also J2.6 (Pin_6), Assr4ch1.A2; no longer J2.3 (Pin_3)
- net A1: no longer names the net of XA1.A1
- net A2: no longer names the net of XA1.A2
- net A3: no longer names the net of XA1.A3
- net A4: no longer names the net of XA1.A4
- net A5: no longer names the net of XA1.A5
- net AGND renamed GNDA
- net GNDA: now also J7.S
- net AREF: no longer names the net of XA1.AREF
- net D10 renamed CamTTL
- net CamTTL: now also J10.2
- net D11 renamed Puff
- net D12 renamed ImagingTrig
- net ImagingTrig: now also J11.2
- net D13: no longer names the net of XA1.D13
- net D2 renamed EncA
- net EncA: now also RotaryEncoder1.1 (A)
- net D3 renamed EncB
- net EncB: now also RotaryEncoder1.2 (B)
- net D4 renamed ShockRelayCh12
- net ShockRelayCh12: now also Assr4ch1.CH1, Assr4ch1.CH2, J1.3 (Pin_3)
- net D5 renamed ShockPWM
- net ShockPWM: now also J2.8 (Pin_8), Assr4ch1.A1; no longer J2.1 (Pin_1)
- net D6 renamed ShockRelayCh34
- net ShockRelayCh34: now also Assr4ch1.CH3, Assr4ch1.CH4, J1.4 (Pin_4)
- net D7 renamed ShockStimIsolator
- net D8 renamed TONE+
- net TONE+: now also J7.T
- net D9 renamed LED
- net RST: no longer names the net of XA1.RST1 (RESET)
- net V_IN: no longer names the net of XA1.VIN
- no-connect marks 15 -> 34
Other:
- note added: "Shock Pad Subcircuit"
- note added: "ShockPad is connected to A0."
- note removed: "CAM\n\n"
- note removed: "Extra pin for new arduino version\n"
- note removed: "For Encoder\n"
- note removed: "Imaging Trig\n"
- note removed: "LED\n"
- note removed: "SSR Relay\n"
- note removed: "Stimulator\n\n"
- note removed: "Tone\n"
- moved on the sheet: C1, D1, J12, J3, J4, J5, J6, J9, Q1, R1, R2, R3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

Commit message: Got a PCB layout.
Parts:
- added J13: StimIsoIN, Connector_Molex:Molex_KK-254_AE-6410-02A_1x02_P2.54mm_Vertical, symbol Connector_Generic:Conn_01x02
Connections:
- net GNDD is gone; now on net GNDA: Assr4ch1.DC-, C1.2, J1.2 (Pin_2), J10.6, J11.6, J4.2 (Ext), J5.2 (Pin_2), J6.2 (Pin_2), J9.2 (Pin_2), R1.2, RotaryEncoder1.4 (GND), U1.2, XA1.GND1 (GND)
- net GNDA: now also J13.1 (Pin_1)
- net ShockStimIsolator: now also J13.2 (Pin_2)
Changed lines of the file:
@@
 Wire Wire Line
 	1225 2950 1400 2950
-Text GLabel 1225 3250 0    60   Input ~ 0
+Text GLabel 1225 3175 0    60   Input ~ 0
 AGND
 $Comp
 L power:GNDA #PWR02
 U 1 1 5D24B4AF
-P 1550 3250
-F 0 "#PWR02" H 1550 3000 50  0001 C CNN
-F 1 "GNDA" V 1555 3122 50  0000 R CNN
-F 2 "" H 1550 3250 50  0001 C CNN
-F 3 "" H 1550 3250 50  0001 C CNN
-	1    1550 3250
+P 1550 3175
+F 0 "#PWR02" H 1550 2925 50  0001 C CNN
+F 1 "GNDA" V 1555 3047 50  0000 R CNN
+F 2 "" H 1550 3175 50  0001 C CNN
+F 3 "" H 1550 3175 50  0001 C CNN
+	1    1550 3175
 	0    -1   -1   0
 $EndComp
-Wire Wire Line
-	1550 3250 1350 3250
 $Comp
 L power:PWR_FLAG #FLG03
@@
 Wire Wire Line
 	1400 2950 1550 2950
-$Comp
-L power:PWR_FLAG #FLG01
-U 1 1 5D24E255
-P 1350 3250
-F 0 "#FLG01" H 1350 3325 50  0001 C CNN
-F 1 "PWR_FLAG" H 1350 3423 50  0000 C CNN
-F 2 "" H 1350 3250 50  0001 C CNN
-F 3 "~" H 1350 3250 50  0001 C CNN
-	1    1350 3250
-	1    0    0    -1
-$EndComp
-Connection ~ 1350 3250
-Wire Wire Line
-	1350 3250 1225 3250
 Text GLabel 1550 3475 2    60   Input ~ 0
 5V
@@
 	1    0    0    -1
 $EndComp
+$Comp
+L Connector_Generic:Conn_01x02 J13
+U 1 1 5D2BFB14
+P 6275 5925
+F 0 "J13" H 6355 5917 50  0000 L CNN
+F 1 "StimIsoIN" H 6355 5826 50  0000 L CNN
+F 2 "Connector_Molex:Molex_KK-254_AE-6410-02A_1x02_P2.54mm_Vertical" H 6275 5925 50  0001 C CNN
+F 3 "~" H 6275 5925 50  0001 C CNN
+	1    6275 5925
+	1    0    0    -1
+$EndComp
+Text GLabel 6075 5925 0    60   Input ~ 0
+DGND
+Text GLabel 6075 6025 0    60   Input ~ 0
+ShockStimIsolator
+Wire Wire Line
+	1225 3175 1400 3175
+Wire Wire Line
+	1400 2950 1400 3175
+Connection ~ 1400 3175
+Wire Wire Line
+	1400 3175 1550 3175
 $EndSCHEMATC
