File: CAD/KiCAD/PreviousVersion/ArduinoEncoderShield_old.sch (KiCad schematic (older format))
At the start: 31 parts, among them CN1 HDR-1X15-15-91-?, IC1 4N25, IC2 4N25, IC3 4N25, IC4 4N25, IC5 4N25, P1 CONN_6, P10 CONN_8, P11 CONN_8, P12 CONN_2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

Commit message: Passing electrical rules.
Parts:
- removed IC3: 4N25, DIP6, symbol 4N25
- removed P2, P3, P4, P5: CONN_2, symbol CONN_2
- added C1: 47 uF, Capacitor_THT:CP_Axial_L11.0mm_D6.0mm_P18.00mm_Horizontal, symbol Device:C
- added IC1: 4N35, Package_DIP:DIP-6_W7.62mm_Socket, symbol Isolator:4N35
- added J-InStimInput1: 90V, Connector_BarrelJack:BarrelJack_CUI_PJ-036AH-SMT_Horizontal, symbol Connector:Jack-DC
- added J1: SSR-ToInput, Connector_PinSocket_2.54mm:PinSocket_1x06_P2.54mm_Vertical, symbol Connector_Generic:Conn_01x06
- added J2: SSR-ToOutput, symbol Connector_Generic:Conn_01x08
- added JPad1: ShockPad, TerminalBlock:TerminalBlock_Altech_AK300-2_P5.00mm, symbol Connector:Screw_Terminal_01x02
- added JPad2: StimInput, TerminalBlock:TerminalBlock_Altech_AK300-2_P5.00mm, symbol Connector:Screw_Terminal_01x02
- added R3: 10k-1M, Potentiometer_THT:Potentiometer_Alps_RK09K_Single_Vertical, symbol Device:R_Variable
- CN1: value HDR-1X15-15-91-? -> OutputPad; footprint con-hdrs40-15-91-15 -> Connector_PinHeader_2.54mm:PinHeader_1x15_P2.54mm_Horizontal; symbol HDR-1X15-15-91-? -> ArduinoEncoderShield_old-rescue:HDR-1X15-15-91-?
- D1: footprint ~ -> Diode_THT:D_5KP_P12.70mm_Horizontal; symbol DIODE -> ArduinoEncoderShield_old-rescue:DIODE
- IC2: renamed from IC1; value 4N25 -> 4N35; footprint DIP6 -> Package_DIP:DIP-6_W7.62mm_Socket; symbol 4N25 -> Isolator:4N35
- IC3: renamed from IC2; value 4N25 -> 4N35; footprint DIP6 -> Package_DIP:DIP-6_W7.62mm_Socket; symbol 4N25 -> Isolator:4N35
- IC4, IC5: value 4N25 -> 4N35; footprint DIP6 -> Package_DIP:DIP-6_W7.62mm_Socket; symbol 4N25 -> Isolator:4N35
- P1: footprint (none) -> Connector_PinHeader_1.27mm:PinHeader_1x06_P1.27mm_Horizontal; symbol CONN_6 -> ArduinoEncoderShield_old-rescue:CONN_6
- P2: renamed from P6; footprint (none) -> Connector_PinHeader_1.27mm:PinHeader_1x06_P1.27mm_Horizontal; symbol CONN_6 -> ArduinoEncoderShield_old-rescue:CONN_6
- P4: renamed from P12; footprint (none) -> Connector_PinHeader_1.27mm:PinHeader_1x02_P1.27mm_Vertical; symbol CONN_2 -> ArduinoEncoderShield_old-rescue:CONN_2
- P7: renamed from P9; symbol CONN_2 -> ArduinoEncoderShield_old-rescue:CONN_2
- P8: renamed from P10; footprint (none) -> Connector_PinHeader_1.27mm:PinHeader_1x08_P1.27mm_Horizontal; symbol CONN_8 -> ArduinoEncoderShield_old-rescue:CONN_8
- P9: renamed from P11; footprint (none) -> Connector_PinHeader_1.27mm:PinHeader_1x08_P1.27mm_Horizontal; symbol CONN_8 -> ArduinoEncoderShield_old-rescue:CONN_8
- R1: renamed from R5; footprint ~ -> Resistor_SMD:R_0603_1608Metric_Pad1.05x0.95mm_HandSolder; symbol R -> ArduinoEncoderShield_old-rescue:R
- R10: renamed from R8; footprint ~ -> Resistor_SMD:R_0805_2012Metric_Pad1.15x1.40mm_HandSolder; symbol R -> ArduinoEncoderShield_old-rescue:R
- R11: footprint ~ -> Resistor_SMD:R_0805_2012Metric_Pad1.15x1.40mm_HandSolder; symbol R -> ArduinoEncoderShield_old-rescue:R
- R12: renamed from R9; footprint ~ -> Resistor_SMD:R_0805_2012Metric_Pad1.15x1.40mm_HandSolder; symbol R -> ArduinoEncoderShield_old-rescue:R
- R13: renamed from R12; footprint ~ -> Resistor_SMD:R_0805_2012Metric_Pad1.15x1.40mm_HandSolder; symbol R -> ArduinoEncoderShield_old-rescue:R
- R2: renamed from R6; footprint ~ -> Resistor_SMD:R_0603_1608Metric_Pad1.05x0.95mm_HandSolder; symbol R -> ArduinoEncoderShield_old-rescue:R
- R4: renamed from R7; footprint ~ -> Resistor_SMD:R_0805_2012Metric_Pad1.15x1.40mm_HandSolder; symbol R -> ArduinoEncoderShield_old-rescue:R
- R5: renamed from R1; footprint ~ -> Resistor_SMD:R_0805_2012Metric_Pad1.15x1.40mm_HandSolder; symbol R -> ArduinoEncoderShield_old-rescue:R
- R6: renamed from R3; footprint ~ -> Resistor_SMD:R_0805_2012Metric_Pad1.15x1.40mm_HandSolder; symbol R -> ArduinoEncoderShield_old-rescue:R
- R7: renamed from R10; footprint ~ -> Resistor_SMD:R_0805_2012Metric_Pad1.15x1.40mm_HandSolder; symbol R -> ArduinoEncoderShield_old-rescue:R
- R8: renamed from R4; footprint ~ -> Resistor_SMD:R_0805_2012Metric_Pad1.15x1.40mm_HandSolder; symbol R -> ArduinoEncoderShield_old-rescue:R
- R9: renamed from R2; footprint ~ -> Resistor_SMD:R_0805_2012Metric_Pad1.15x1.40mm_HandSolder; symbol R -> ArduinoEncoderShield_old-rescue:R
- SHIELD1: symbol ARDUINO_SHIELD -> ArduinoEncoderShield_old-rescue:ARDUINO_SHIELD
- U1: footprint (none) -> Package_DIP:DIP-16_W7.62mm_Socket; symbol ULN2003A -> ArduinoEncoderShield_old-rescue:ULN2003A
Connections:
- net 5V: now also J1.1 (Pin_1)
- net A0: now also C1.1, J2.6 (Pin_6), R3.1
- net AGND: now also SHIELD1.GND1, C1.2, R3.2
- net D4: now also J1.3 (Pin_3), J1.4 (Pin_4)
- net D5: now also J2.8 (Pin_8)
- net D6: now also J1.5 (Pin_5), J1.6 (Pin_6)
- net D7: now also JPad2.1 (Pin_1)
- net DGND: now also IC1.2, J1.2 (Pin_2), JPad2.2 (Pin_2); no longer SHIELD1.GND1, SHIELD1.GND2, SHIELD1.GND3
- net EX 5 V: now also IC1.5
- net Tone3: now also IC1.4
- net at R4.2: now also IC1.1
- net 3V3: no longer names the net of SHIELD1.3V3
- net 3V3: no longer P1.5
- net AREF: no longer names the net of SHIELD1.AREF
- net AREF: no longer P9.1 (P1)
- net V_IN: no longer names the net of SHIELD1.V_IN
- net V_IN: no longer P1.1
- new net: J-InStimInput1.1, J2.2 (Pin_2)
- new net: J-InStimInput1.2, J2.4 (Pin_4)
- new net: J2.1 (Pin_1), J2.5 (Pin_5), JPad1.2 (Pin_2)
- new net: J2.3 (Pin_3), J2.7 (Pin_7), JPad1.1 (Pin_1)
- no-connect marks 0 -> 23
Other:
- moved on the sheet: D1, P8, P9, R10, R11, R12, R13, R4, R5, R6, R7, R8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
